Commit message: chore: R2D2 bot passes navigation test! expanded inflation_radius, corrected wheel separation, and slowed down movement.

File: urdf/my_bot.xacro (robot description, xacro)
@@ -12,5 +12,5 @@
     <pose>0 0 0.1 0 0 0</pose>
     <inertial>
-      <mass value="15.0"/>
+      <mass value="2.0"/>
       <origin xyz="0.0 0 0" rpy=" 0 0 0"/>
       <inertia
